Commit message: fix: 修正激光传感器的旋转角度为 3.14159

File: src/vehicle_bringup/description/vehicle.urdf (robot description, URDF)
Before this commit: robot bunker_bot, 4 links, 3 joints
Joints:
- joint base_to_laser: origin xyz=0.2 0.0 0.15 rpy=0 0 0 -> xyz=0.2 0.0 0.15 rpy=0 0 3.14159

Commit message: fix: 调整地图更新间隔和激光传感器的旋转角度，修正IMU连接位置

File: src/vehicle_bringup/description/vehicle.urdf (robot description, URDF)
Before this commit: robot bunker_bot, 4 links, 3 joints
Joints:
- joint base_to_imu: origin xyz=0.0 0.0 0.1 rpy=0 0 0 -> xyz=-0.2 -0.15 0.15 rpy=0 0 0
- joint base_to_laser: origin xyz=0.2 0.0 0.15 rpy=0 0 3.14159 -> xyz=0.2 0.0 0.15 rpy=-0 0 3.1415926
